Commit message: Initial commit: qua_engineer training complement using robot_lab

File: source/robot_lab/data/Robots/unitree/go2_description/urdf/go2_description.urdf (robot description, URDF)
Before this commit: robot go2_description, 42 links, 41 joints
Links:
- added link left_arm1, mass 0.515038; visual mesh filename=../meshes/left_arm1.STL
- added link left_arm2, mass 0.266875; visual mesh filename=../meshes/left_arm2.STL
- added link left_arm3, mass 2.186092; visual mesh filename=../meshes/left_arm3.STL
- added link right_arm1, mass 0.515038; visual mesh filename=../meshes/right_arm1.STL
- added link right_arm2, mass 0.266875; visual mesh filename=../meshes/right_arm2.STL
- added link right_arm3, mass 2.186092; visual mesh filename=../meshes/right_arm3.STL
- link FL_calf: mass 0.154 -> 0.195
- link FL_hip: mass 0.678 -> 1.069
- link FL_thigh: mass 1.152 -> 1.257
- link FR_calf: mass 0.154 -> 0.195
- link FR_hip: mass 0.678 -> 1.069
- link FR_thigh: mass 1.152 -> 1.257
- link RL_calf: mass 0.154 -> 0.194642
- link RL_hip: mass 0.678 -> 1.069477
- link RL_thigh: mass 1.152 -> 1.256985
- link RR_calf: mass 0.154 -> 0.194642
- link RR_hip: mass 0.678 -> 1.069477
- link RR_thigh: mass 1.152 -> 1.256985
- link base: mass 6.921 -> 14.140726; geometry collision box size=0.1 0.1 0.1; collision box size=0.1 0.1 0.1
Joints:
- added joint left_arm_j1: type fixed, parent base, child left_arm1, origin xyz=0.1 -0.085 0.05 rpy=0 0 -1.5708, axis 0 0 0
- added joint left_arm_j2: type fixed, parent left_arm1, child left_arm2, origin xyz=0 0.038 0.036 rpy=-1.5708 0 0, axis 0 0 0
- added joint left_arm_j3: type fixed, parent left_arm2, child left_arm3, origin xyz=-0.2388 0 -0.009 rpy=3.1416 0 0, axis 0 0 0
- added joint right_arm_j1: type fixed, parent base, child right_arm1, origin xyz=-0.1 -0.085 0.05 rpy=0 0 -1.5708, axis 0 0 0
- added joint right_arm_j2: type fixed, parent right_arm1, child right_arm2, origin xyz=0 -0.038 0.036 rpy=1.5708 0 0, axis 0 0 0
- added joint right_arm_j3: type fixed, parent right_arm2, child right_arm3, origin xyz=-0.2388 0 -0.009 rpy=-3.1416 0 0, axis 0 0 0
- joint FL_calf_joint: limit lower=-2.7227 upper=-0.83776 effort=45.43 velocity=15.70 -> lower=-3.2 upper=3.2 effort=45.43 velocity=15.70
- joint FL_hip_joint: limit lower=-1.0472 upper=1.0472 effort=23.7 velocity=30.1 -> lower=-1.00 upper=0.50 effort=23.7 velocity=30.1
- joint FL_thigh_joint: limit lower=-1.5708 upper=3.4907 effort=23.7 velocity=30.1 -> lower=-3.2 upper=3.2 effort=23.7 velocity=30.1
- joint FR_calf_joint: limit lower=-2.7227 upper=-0.83776 effort=45.43 velocity=15.70 -> lower=-3.2 upper=3.2 effort=45.43 velocity=15.70
- joint FR_hip_joint: limit lower=-1.0472 upper=1.0472 effort=23.7 velocity=30.1 -> lower=-0.50 upper=1.00 effort=23.7 velocity=30.1
- joint FR_thigh_joint: limit lower=-1.5708 upper=3.4907 effort=23.7 velocity=30.1 -> lower=-3.2 upper=3.2 effort=23.7 velocity=30.1
- joint RL_calf_joint: limit lower=-2.7227 upper=-0.83776 effort=45.43 velocity=15.70 -> lower=-3.2 upper=3.2 effort=45.43 velocity=15.70
- joint RL_hip_joint: limit lower=-1.0472 upper=1.0472 effort=23.7 velocity=30.1 -> lower=-1.00 upper=0.50 effort=23.7 velocity=30.1
- joint RL_thigh_joint: limit lower=-0.5236 upper=4.5379 effort=23.7 velocity=30.1 -> lower=-3.2 upper=3.2 effort=23.7 velocity=30.1
- joint RR_calf_joint: limit lower=-2.7227 upper=-0.83776 effort=45.43 velocity=15.70 -> lower=-3.2 upper=3.2 effort=45.43 velocity=15.70
- joint RR_hip_joint: limit lower=-1.0472 upper=1.0472 effort=23.7 velocity=30.1 -> lower=-0.50 upper=1.00 effort=23.7 velocity=30.1
- joint RR_thigh_joint: limit lower=-0.5236 upper=4.5379 effort=23.7 velocity=30.1 -> lower=-3.2 upper=3.2 effort=23.7 velocity=30.1
